Commit message: try lab4

File: install/task2/share/task2/urdf/base_ns.urdf.xacro (robot description, xacro)
@@ -44,5 +44,5 @@
         </link>
         <!-- 机器人关节 -->
-        <joint name="${namespace}_joint_name" type="fixed">
+        <joint name="${namespace}/joint_name" type="fixed">
             <!-- 父部件 -->
             <parent link="${namespace}/base_footprint" />

File: install/task2/share/task2/urdf/common_inertia_ns.xacro (robot description, xacro)
@@ -3,5 +3,5 @@
     <!-- 定义命名空间参数 -->
     <xacro:arg name="namespace" default="default_ns"/>
-    <xacro:macro name="${namespace}_box_inertia" params="m w h d">
+    <xacro:macro name="${namespace}/box_inertia" params="m w h d">
         <inertial>
             <mass value="${m}" />
@@ -9,5 +9,5 @@
         </inertial>
     </xacro:macro>
-    <xacro:macro name="${namespace}_cylinder_inertia" params="m r h">
+    <xacro:macro name="${namespace}/cylinder_inertia" params="m r h">
         <inertial>
             <mass value="${m}" />
@@ -15,5 +15,5 @@
         </inertial>
     </xacro:macro>
-    <xacro:macro name="${namespace}_sphere_inertia" params="m r">
+    <xacro:macro name="${namespace}/sphere_inertia" params="m r">
         <inertial>
             <mass value="${m}" />

File: install/task2/share/task2/urdf/plugins/gazebo_sensor_plugin_ns.xacro (robot description, xacro)
@@ -3,7 +3,7 @@
     <xacro:macro name="gazebo_sensor_plugin" params="namespace">
         <!-- 激光传感器 -->
-        <gazebo reference="laser_link">
-            <sensor name="${namespace}_laserscan" type="ray">
-                <plugin name="${namespace}_laserscan_plugin" filename="libgazebo_ros_ray_sensor.so">
+        <gazebo reference="${namespace}/laser_link">
+            <sensor name="${namespace}/laserscan" type="ray">
+                <plugin name="laserscan_plugin" filename="libgazebo_ros_ray_sensor.so">
                     <ros>
                         <namespace>${namespace}</namespace>
@@ -11,5 +11,5 @@
                     </ros>
                     <output_type>sensor_msgs/LaserScan</output_type>
-                    <frame_name>laser_link</frame_name>
+                    <frame_name>${namespace}/laser_link</frame_name>
                 </plugin>
                 <always_on>true</always_on>
@@ -40,10 +40,10 @@
         </gazebo>
         <!-- IMU 传感器 -->
-        <gazebo reference="imu_link">
-            <sensor name="${namespace}_imu_sensor" type="imu">
-                <plugin name="${namespace}_imu_plugin" filename="libgazebo_ros_imu_sensor.so">
+        <gazebo reference="${namespace}/imu_link">
+            <sensor name="${namespace}/imu_sensor" type="imu">
+                <plugin name="imu_plugin" filename="libgazebo_ros_imu_sensor.so">
                     <ros>
                         <namespace>${namespace}</namespace>
-                        <remapping>~/out:=${namespace}/imu</remapping>
+                        <remapping>~/out:=imu</remapping>
                     </ros>
                     <initial_orientation_as_reference>false</initial_orientation_as_reference>
@@ -108,7 +108,7 @@
         </gazebo>
         <!-- 深度相机 -->
-        <gazebo reference="camera_link">
-            <sensor type="depth" name="${namespace}_camera_sensor">
-                <plugin name="${namespace}_depth_camera" filename="libgazebo_ros_camera.so">
+        <gazebo reference="${namespace}/camera_link">
+            <sensor type="depth" name="${namespace}/camera_sensor">
+                <plugin name="depth_camera" filename="libgazebo_ros_camera.so">
                     <ros>
                         <namespace>${namespace}</namespace>
@@ -118,5 +118,5 @@
                 <always_on>true</always_on>
                 <update_rate>10</update_rate>
-                <camera name="camera">
+                <camera name="${namespace}/camera">
                     <horizontal_fov>1.5009831567</horizontal_fov>
                     <image>

File: install/task2/share/task2/urdf/sensor/camera_ns.urdf.xacro (robot description, xacro)
@@ -7,7 +7,7 @@
     <xacro:macro name="camera_xacro" params="namespace xyz">
         <!-- 虚拟模块 -->
-        <link name="${namespace}_camera_optical_link"></link>
+        <link name="${namespace}/camera_optical_link"></link>
         <!-- 机器人 IMU 部件 -->
-        <link name="${namespace}_camera_link">
+        <link name="${namespace}/camera_link">
             <visual>
                 <origin xyz="0 0 0" rpy="0 0 0" />
@@ -31,20 +31,20 @@
         </link>
         <!-- 机器人关节 -->
-        <joint name="${namespace}_camera_joint" type="fixed">
+        <joint name="${namespace}/camera_joint" type="fixed">
             <!-- 父部件 -->
             <parent link="${namespace}/base_link" />
             <!-- 子部件 -->
-            <child link="${namespace}_camera_link" />
+            <child link="${namespace}/camera_link" />
             <!-- 子部件相对父部件的平移和旋转 -->
             <origin xyz="${xyz}" rpy="0 0 0" />
         </joint>
         <!-- 把相机 z 轴朝向前方 -->
-        <joint name="${namespace}_camera_optical_link_joint" type="fixed">
-            <parent link="${namespace}_camera_link" />
-            <child link="${namespace}_camera_optical_link" />
+        <joint name="${namespace}/camera_optical_link_joint" type="fixed">
+            <parent link="${namespace}/camera_link" />
+            <child link="${namespace}/camera_optical_link" />
             <origin xyz="0 0 0" rpy="${-pi/2} 0.0 ${-pi/2}" />
         </joint>
         <!-- Gazebo 配置 -->
-        <gazebo reference="${namespace}_camera_link">
+        <gazebo reference="${namespace}/camera_link">
             <material>Gazebo/Yellow</material>
         </gazebo>

File: install/task2/share/task2/urdf/sensor/imu_ns.urdf.xacro (robot description, xacro)
@@ -7,5 +7,5 @@
     <xacro:macro name="imu_xacro" params="namespace xyz">
         <!-- 机器人IMU部件 -->
-        <link name="${namespace}_imu_link">
+        <link name="${namespace}/imu_link">
             <visual>
                 <origin xyz="0 0 0" rpy="0 0 0" />
@@ -29,9 +29,9 @@
         </link>
         <!-- 机器人关节 -->
-        <joint name="${namespace}_imu_joint" type="fixed">
+        <joint name="${namespace}/imu_joint" type="fixed">
             <!-- 父部件 -->
             <parent link="${namespace}/base_link" />
             <!-- 子部件 -->
-            <child link="${namespace}_imu_link" />
+            <child link="${namespace}/imu_link" />
             <!-- 子部件相对父部件的平移和旋转 -->
             <origin xyz="${xyz}" rpy="0 0 0" />

File: install/task2/share/task2/urdf/sensor/laser_ns.urdf.xacro (robot description, xacro)
@@ -7,5 +7,5 @@
     <xacro:macro name="laser_xacro" params="namespace xyz">
         <!-- 雷达支撑杆 -->
-        <link name="${namespace}_laser_cylinder_link">
+        <link name="${namespace}/laser_cylinder_link">
             <visual>
                 <origin xyz="0 0 0" rpy="0 0 0" />
@@ -29,5 +29,5 @@
         </link>
         <!-- 雷达 -->
-        <link name="${namespace}_laser_link">
+        <link name="${namespace}/laser_link">
             <visual>
                 <origin xyz="0 0 0" rpy="0 0 0" />
@@ -51,24 +51,24 @@
         </link>
         <!-- 将雷达固定到支撑杆 -->
-        <joint name="${namespace}_laser_joint" type="fixed">
+        <joint name="${namespace}/laser_joint" type="fixed">
             <!-- 父部件 -->
-            <parent link="${namespace}_laser_cylinder_link" />
+            <parent link="${namespace}/laser_cylinder_link" />
             <!-- 子部件 -->
-            <child link="${namespace}_laser_link" />
+            <child link="${namespace}/laser_link" />
             <!-- 子部件相对父部件的平移和旋转 -->
             <origin xyz="0 0 0.05" rpy="0 0 0" />
         </joint>
-        <joint name="${namespace}_laser_cylinder_joint" type="fixed">
+        <joint name="${namespace}/laser_cylinder_joint" type="fixed">
             <!-- 父部件 -->
             <parent link="${namespace}/base_link" />
             <!-- 子部件 -->
-            <child link="${namespace}_laser_cylinder_link" />
+            <child link="${namespace}/laser_cylinder_link" />
             <!-- 子部件相对父部件的平移和旋转 -->
             <origin xyz="${xyz}" rpy="0 0 0" />
         </joint>
-        <gazebo reference="${namespace}_laser_cylinder_link">
+        <gazebo reference="${namespace}/laser_cylinder_link">
             <material>Gazebo/Red</material>
         </gazebo>
-        <gazebo reference="${namespace}_laser_link">
+        <gazebo reference="${namespace}/laser_link">
             <material>Gazebo/Red</material>
         </gazebo>
